File: hardware/tempsensor_project/tempsensor_project.kicad_sch (KiCad schematic)
At the start: 2 parts, among them U1 PIC18F4520-xP

Commit message: updated schematic
Parts:
- added U2: TC74A5-5.0VAT, TO-220_AT_MC_MCH, symbol finalproject:TC74A5-5.0VAT
Changed lines of the file:
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@@
+    )
+  )
+  (symbol (lib_id "finalproject:TC74A5-5.0VAT") (at 142.24 113.03 0) (unit 1)
+    (in_bom yes) (on_board yes) (dnp no) (fields_autoplaced)
+    (property "Reference" "U2" (at 170.18 104.14 0)
+      (effects (font (size 1.524 1.524)))
+    )
+    (property "Value" "TC74A5-5.0VAT" (at 170.18 106.68 0)
+      (effects (font (size 1.524 1.524)))
+    )
+    (property "Footprint" "TO-220_AT_MC_MCH" (at 142.24 113.03 0)
+      (effects (font (size 1.27 1.27) italic) hide)
+    )
+    (property "Datasheet" "TC74A5-5.0VAT" (at 142.24 113.03 0)
+      (effects (font (size 1.27 1.27) italic) hide)
+    )
+    (pin "1")
+    (pin "2")
+    (pin "3")
+    (pin "4")
+    (pin "5")
+    (instances
+      (project "tempsensor_project"
+        (path "/3fe1aeb8-57a5-41c7-b00d-11c7bf39123b"
+          (reference "U2") (unit 1)
+        )
+      )
     )
   )

Commit message: updated schematic
Parts:
- added SW1: SW_SPST, symbol Switch:SW_SPST
Connections:
- net +5V: now reaches U1.11 (VDD), U1.32 (VDD)
- net +5V: now also DS1.4 (VDD), U2.5 (VDD), SW1.1 (A)
- net Earth: now reaches U1.12 (VSS), U1.31 (VSS)
- net Earth: now also DS1.3 (VSS), U2.3 (GND)
- net at U1.15 (RC0): now also DS1.6 (RS)
- net at U1.16 (RC1): now also DS1.7 (R/~{W})
- net at U1.18 (RC3): now also U2.4 (SCLK)
- net at U1.19 (RD0): now also DS1.9 (DB0)
- net at U1.20 (RD1): now also DS1.10 (DB1)
- net at U1.21 (RD2): now also DS1.11 (DB2)
- net at U1.22 (RD3): now also DS1.12 (DB3)
- net at U1.23 (RC4): now also U2.2 (SDA)
- net at U1.27 (RD4): now also DS1.13 (DB4)
- net at U1.28 (RD5): now also DS1.14 (DB5)
- net at U1.29 (RD6): now also DS1.15 (DB6)
- net at U1.30 (RD7): now also DS1.16 (DB7)
- net at U1.33 (RB0): now also SW1.2 (B)
Other:
- company: (none) -> UD EMST
- title: (none) -> Temperature Sensor Project
- moved on the sheet: DS1
